File: kicad/glutte-coulombcounter.kicad_pcb (KiCad board)
At the start: 2 copper layers, 100 x 85 mm, 70 parts, among them J1 12V, J2 Measure, J3 K1, J4 AVR-ISP-6, J5 Glutte, J6 K2, J7 K3, J8 Raspi, K1 G6SK-2F-DC5, K2 G6SK-2F-DC5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

Commit message: Add pullups on CSn and UART TX
Parts:
- added R16: 4k7, Resistor_SMD:R_1206_3216Metric_Pad1.42x1.75mm_HandSolder, F.Cu at (73.2, 35.6)
- added R17: 4k7, Resistor_SMD:R_1206_3216Metric_Pad1.42x1.75mm_HandSolder, F.Cu at (68.1, 85.9)
Routing:
- net /SSn: track 42.2 -> 50.1 mm
- net /TXD: track 38.6 -> 42.3 mm
- net +5VA: track 388.4 -> 390.6 mm, vias 5 -> 6
Changed lines of the file:
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@@
     (thickness 1.6)
     (drawings 130)
-    (tracks 785)
+    (tracks 795)
     (zones 0)
-    (modules 70)
+    (modules 72)
     (nets 82)
   )
@@
   )
   (setup
-    (last_trace_width 0.2)
+    (last_trace_width 0.25)
     (user_trace_width 0.2)
     (user_trace_width 0.25)
@@
     (add_net "Net-(J7-Pad6)")
   )
+  (module Resistor_SMD:R_1206_3216Metric_Pad1.42x1.75mm_HandSolder (layer F.Cu)
+    (at 68.072 85.852 180)
+    (descr "Resistor SMD 1206 (3216 Metric), square (rectangular) end terminal, IPC_7351 nominal with elongated pad for handsoldering. (Body size source: http://www.tortai-tech.com/upload/download/2011102023233369053.pdf), generated with kicad-footprint-generator")
+    (tags "resistor handsolder")
+    (attr smd)
+    (fp_text reference R17 (at -0.508 -1.82) (layer F.SilkS)
+      (effects (font (size 1 1) (thickness 0.15)))
+    )
+    (fp_text value 4k7 (at 0 1.82) (layer F.Fab)
+      (effects (font (size 1 1) (thickness 0.15)))
+    )
+    (fp_text user %R (at 0 0) (layer F.Fab)
+      (effects (font (size 0.8 0.8) (thickness 0.12)))
+    )
+    (fp_line (start 2.45 1.12) (end -2.45 1.12) (layer F.CrtYd) (width 0.05))
+    (fp_line (start 2.45 -1.12) (end 2.45 1.12) (layer F.CrtYd) (width 0.05))
+    (fp_line (start -2.45 -1.12) (end 2.45 -1.12) (layer F.CrtYd) (width 0.05))
+    (fp_line (start -2.45 1.12) (end -2.45 -1.12) (layer F.CrtYd) (width 0.05))
+    (fp_line (start -0.602064 0.91) (end 0.602064 0.91) (layer F.SilkS) (width 0.12))
+    (fp_line (start -0.602064 -0.91) (end 0.602064 -0.91) (layer F.SilkS) (width 0.12))
+    (fp_line (start 1.6 0.8) (end -1.6 0.8) (layer F.Fab) (width 0.1))
+    (fp_line (start 1.6 -0.8) (end 1.6 0.8) (layer F.Fab) (width 0.1))
+    (fp_line (start -1.6 -0.8) (end 1.6 -0.8) (layer F.Fab) (width 0.1))
+    (fp_line (start -1.6 0.8) (end -1.6 -0.8) (layer F.Fab) (width 0.1))
+    (pad 2 smd roundrect (at 1.4875 0 180) (size 1.425 1.75) (layers F.Cu F.Paste F.Mask) (roundrect_rratio 0.175439)
+      (net 6 +5VA))
+    (pad 1 smd roundrect (at -1.4875 0 180) (size 1.425 1.75) (layers F.Cu F.Paste F.Mask) (roundrect_rratio 0.175439)
+      (net 43 /TXD))
+    (model ${KISYS3DMOD}/Resistor_SMD.3dshapes/R_1206_3216Metric.wrl
+      (at (xyz 0 0 0))
+      (scale (xyz 1 1 1))
+      (rotate (xyz 0 0 0))
+    )
+  )
+  (module Resistor_SMD:R_1206_3216Metric_Pad1.42x1.75mm_HandSolder (layer F.Cu)
+    (at 73.152 35.56 90)
+    (descr "Resistor SMD 1206 (3216 Metric), square (rectangular) end terminal, IPC_7351 nominal with elongated pad for handsoldering. (Body size source: http://www.tortai-tech.com/upload/download/2011102023233369053.pdf), generated with kicad-footprint-generator")
+    (tags "resistor handsolder")
+    (attr smd)
+    (fp_text reference R16 (at 0 -1.82 90) (layer F.SilkS)
+      (effects (font (size 1 1) (thickness 0.15)))
+    )
+    (fp_text value 4k7 (at 0 1.82 90) (layer F.Fab)
+      (effects (font (size 1 1) (thickness 0.15)))
+    )
+    (fp_text user %R (at 0 0 90) (layer F.Fab)
+      (effects (font (size 0.8 0.8) (thickness 0.12)))
+    )
+    (fp_line (start 2.45 1.12) (end -2.45 1.12) (layer F.CrtYd) (width 0.05))
+    (fp_line (start 2.45 -1.12) (end 2.45 1.12) (layer F.CrtYd) (width 0.05))
+    (fp_line (start -2.45 -1.12) (end 2.45 -1.12) (layer F.CrtYd) (width 0.05))
+    (fp_line (start -2.45 1.12) (end -2.45 -1.12) (layer F.CrtYd) (width 0.05))
+    (fp_line (start -0.602064 0.91) (end 0.602064 0.91) (layer F.SilkS) (width 0.12))
+    (fp_line (start -0.602064 -0.91) (end 0.602064 -0.91) (layer F.SilkS) (width 0.12))
+    (fp_line (start 1.6 0.8) (end -1.6 0.8) (layer F.Fab) (width 0.1))
+    (fp_line (start 1.6 -0.8) (end 1.6 0.8) (layer F.Fab) (width 0.1))
+    (fp_line (start -1.6 -0.8) (end 1.6 -0.8) (layer F.Fab) (width 0.1))
+    (fp_line (start -1.6 0.8) (end -1.6 -0.8) (layer F.Fab) (width 0.1))
+    (pad 2 smd roundrect (at 1.4875 0 90) (size 1.425 1.75) (layers F.Cu F.Paste F.Mask) (roundrect_rratio 0.175439)
+      (net 38 /SSn))
+    (pad 1 smd roundrect (at -1.4875 0 90) (size 1.425 1.75) (layers F.Cu F.Paste F.Mask) (roundrect_rratio 0.175439)
+      (net 6 +5VA))
+    (model ${KISYS3DMOD}/Resistor_SMD.3dshapes/R_1206_3216Metric.wrl
+      (at (xyz 0 0 0))
+      (scale (xyz 1 1 1))
+      (rotate (xyz 0 0 0))
+    )
+  )
   (module Resistor_THT:R_Array_SIP7 (layer F.Cu)
     (at 118.5545 24.5745 180)
@@
   (segment (start 70.852282 91.844272) (end 71.252281 92.244271) (width 0.4) (layer B.Cu) (net 6))
   (segment (start 71.351552 92.145) (end 71.252281 92.244271) (width 0.4) (layer F.Cu) (net 6))
-  (segment (start 54.032 88.022) (end 67.03001 88.022) (width 0.4) (layer B.Cu) (net 6))
   (segment (start 67.03001 88.022) (end 70.852282 91.844272) (width 0.4) (layer B.Cu) (net 6))
   (segment (start 73.243 92.145) (end 71.351552 92.145) (width 0.4) (layer F.Cu) (net 6))
@@
   (segment (start 98.0075 35.2925) (end 98.0075 27.94) (width 0.4) (layer F.Cu) (net 6))
   (segment (start 100.3575 37.6425) (end 98.0075 35.2925) (width 0.4) (layer F.Cu) (net 6))
+  (via (at 66.686 88.022) (size 0.8) (drill 0.4) (layers F.Cu B.Cu) (net 6))
+  (segment (start 66.5845 87.9205) (end 66.686 88.022) (width 0.25) (layer F.Cu) (net 6))
+  (segment (start 66.5845 85.852) (end 66.5845 87.9205) (width 0.25) (layer F.Cu) (net 6))
+  (segment (start 54.032 88.022) (end 66.686 88.022) (width 0.4) (layer B.Cu) (net 6))
+  (segment (start 66.686 88.022) (end 67.03001 88.022) (width 0.4) (layer B.Cu) (net 6))
   (segment (start 50.4775 61.7) (end 50.8 61.3775) (width 0.4) (layer F.Cu) (net 7))
   (segment (start 46.99 61.7) (end 50.4775 61.7) (width 0.4) (layer F.Cu) (net 7))
@@
   (segment (start 77.28802 64.77) (end 80.580034 61.477986) (width 0.25) (layer F.Cu) (net 38))
   (segment (start 80.580034 61.477986) (end 80.580034 32.955034) (width 0.25) (layer F.Cu) (net 38))
+  (segment (start 79.390067 34.145001) (end 80.580034 32.955034) (width 0.25) (layer F.Cu) (net 38))
+  (segment (start 74.199501 34.145001) (end 79.390067 34.145001) (width 0.25) (layer F.Cu) (net 38))
+  (segment (start 74.127 34.0725) (end 74.199501 34.145001) (width 0.25) (layer F.Cu) (net 38))
+  (segment (start 73.152 34.0725) (end 74.127 34.0725) (width 0.25) (layer F.Cu) (net 38))
   (segment (start 55.691 53.086) (end 55.691 51.816) (width 0.25) (layer F.Cu) (net 39))
   (segment (start 60.641 45.466) (end 60.641 46.736) (width 0.25) (layer F.Cu) (net 40))
@@
   (segment (start 85.725 55.88) (end 83.621032 57.983968) (width 0.25) (layer F.Cu) (net 43))
   (segment (start 83.621032 57.983968) (end 83.621032 73.858968) (width 0.25) (layer F.Cu) (net 43))
+  (segment (start 69.6165 85.795) (end 69.5595 85.852) (width 0.25) (layer F.Cu) (net 43))
+  (segment (start 73.243 85.795) (end 69.6165 85.795) (width 0.25) (layer F.Cu) (net 43))
   (segment (start 86.36 57.785) (end 85.725 58.42) (width 0.25) (layer F.Cu) (net 44))
   (segment (start 85.725 58.42) (end 84.071043 60.073957) (width 0.25) (layer F.Cu) (net 44))
